Commit message: first commit

File: src/learning/robot_sim_lsy/urdf/4wd_test.urdf (robot description, URDF)
Before this commit: robot 4wd_test, 9 links, 8 joints
Links:
- removed link laser_link
- added link gps_link; visual cylinder length=0.01 radius=0.03
- added link imu_link, mass 0.1; visual cylinder length=0.01 radius=0.03
- link dummy_link: mass 100 -> 10
- link left_back_wheel_link: mass 0.1 -> 0.5
- link left_front_wheel_link: mass 0.1 -> 0.5
- link right_back_wheel_link: mass 0.1 -> 0.5
- link right_front_wheel_link: mass 0.1 -> 0.5
Joints:
- removed joint laser_joint
- added joint gps_joint: type fixed, parent base_link, child gps_link, origin xyz=0 0 0.09 rpy=0 0 0
- added joint imu_joint: type fixed, parent base_link, child imu_link, origin xyz=0 0 0.08 rpy=0 0 0
